File: KiCad_Files/USB_Reader.sch (KiCad schematic (older format))
At the start: 27 parts, among them P1 CONN_02X05, P2 USB_A, U1 LM1117_3V3, U2 74HC4050, U3 MAX3421E, Y1 12 MHz

Commit message: Changed value of C5 and C7 to 18pF.
Parts:
- C5, C7: value 20pF -> 18pF
Other:
- note added: "REV. A Initial Prototype"
- note added: "REV. B Changed value of C5 and C7 from 20pF to 18pF.\nBOM Updated, board remains REV. B."
- note added: "REV. B Removed R2 from prototype design and\nrenumbered components."
- note added: "REVISION HISTORY"
Changed lines of the file:
@@
 P 7350 1200
 F 0 "C7" V 7550 1150 50  0000 L CNN
-F 1 "20pF" V 7200 1100 50  0000 L CNN
+F 1 "18pF" V 7200 1100 50  0000 L CNN
 F 2 "Capacitors_SMD:C_0603_HandSoldering" H 7388 1050 50  0001 C CNN
 F 3 "" H 7350 1200 50  0000 C CNN
@@
 P 6350 1200
 F 0 "C5" V 6550 1150 50  0000 L CNN
-F 1 "20pF" V 6200 1100 50  0000 L CNN
+F 1 "18pF" V 6200 1100 50  0000 L CNN
 F 2 "Capacitors_SMD:C_0603_HandSoldering" H 6388 1050 50  0001 C CNN
 F 3 "" H 6350 1200 50  0000 C CNN
@@
 NoConn ~ 6500 3450
 NoConn ~ 2800 3400
+Text Notes 8000 5000 0    60   ~ 0
+REVISION HISTORY
+Text Notes 8000 5200 0    60   ~ 0
+REV. A  Initial Prototype
+Text Notes 8000 5500 0    60   ~ 0
+REV. B  Removed R2 from prototype design and\nrenumbered components.
+Text Notes 8000 5750 0    60   ~ 0
+REV. B  Changed value of C5 and C7 from 20pF to 18pF.\nBOM Updated, board remains REV. B.
 $EndSCHEMATC
