File: KiCad_Files/USB_Reader_Rev_C.sch (KiCad schematic (older format))
At the start: 27 parts, among them P1 CONN_02X05, P2 USB_A, U1 LM1117_3V3, U2 74HC4050, U3 MAX3421E, Y1 12 MHz

Commit message: All board files updated to Rev. C
Parts:
- removed C5: 20pF, Capacitors_SMD:C_0603_HandSoldering, symbol C
- removed U1: LM1117_3V3, TO_SOT_Packages_SMD:TO-252-2Lead, symbol LM1117_3V3
- removed Y1: 12 MHz, AO_Parts:FA-328_Crystal, symbol Crystal_GND24
- added C2: 0.1uF, Capacitors_SMD:C_0603_HandSoldering, symbol C
- added OSC1: Oscillator, AO_Parts:FA-328_Crystal, symbol Oscillator
- added R1: 100k, Resistors_SMD:R_0603_HandSoldering, symbol R
- added R4: 10k, Resistors_SMD:R_0603_HandSoldering, symbol R
- added U1: TLV75533, TO_SOT_Packages_SMD:SOT-23-5, symbol TLV75533
- C7: value 20pF -> 0.1uF
- renumbered C2 to C3, C3 to C4, C4 to C5, R1 to R2, R2 to R3, R3 to R5, R4 to R6, R5 to R7
Connections:
- net +3V3: now also C7.1, OSC1.4 (Vdd), R4.1, U1.5 (Vo)
- net +5V: now also R1.1, U1.1 (Vi)
- net GND: now also C7.2, C2.2, OSC1.2 (GND), U1.2 (GND); no longer C7.1
- net at U3.24 (XI): now also OSC1.3 (OUT); no longer C7.2
- new net: OSC1.1 (SB), R4.2
- new net: C2.1, R1.2, U1.3 (EN)
- no-connect marks 21 -> 23
Other:
- note added: "1) Crystal replaced with 12 MHz MEMS Oscillator Module."
- note added: "12.00 MHz"
- note added: "2) Connector P1 rotated 180 degrees to match ribbon cable."
- note added: "3) Linear Voltage Regulator replaced with TLV75533."
- note added: "4) Delay added to 3.3V supply for faster rise time."
- note added: "P1 USB Reader\n 1 +5V\n 2 GND\n 3 RES\n 4 INT\n 5 MOSI\n 6 N/C\n 7 SS\n 8 N/C\n 9 SCK\n10 MISO"
- note added: "REV. C"
- note added: "SC2 Pinout Archim SAM3X\n 1 +5V\n 2 GND\n 3 NRST\n 4 TIOA0 - PB25\n 5 MOSI - PA26\n 6 TIOB1 - PA3\n 7 CS - PA29\n 8 TIOB0 - PB27\n 9 SCLK - PA27\n10 MISO - PA25"
- note removed: "NOTE - +5V Must be provided\nby an external source as Pin-1\non Archim is +3.3V and Pin-1\non Einsy is connected to PC5."
- note removed: "NOTE - On the Archim schematic, the pin\nnumbers of SC2 (J13) are reversed as\nfollows:\n\nOn Archim Schematic On USB Reader Schematic\nPin-10 Pin-1\nPin-9 Pin-2\nPin-8 Pin-3\nPin-7 Pin-4\nPin-6 Pin-5\nPin-5 Pin-6\nPin-4 Pin-7\nPin-3 Pin-8\nPin-2 Pin-9\nPin-1 Pin-10"
- note removed: "P1 USB Reader\n 1 +5V\n 2 GND\n 3 RES\n 4 INT\n 5 MOSI\n 6 N/C\n 7 SS\n 8 GPX\n 9 SCK\n10 MISO"
- note removed: "P2 Pinout Archim SAM3X\n 1 +3.3V\n 2 GND\n 3 NRST\n 4 TIOA0 - PB25\n 5 MOSI - PA26\n 6 TIOB1 - PA3\n 7 CS - PA29\n 8 TIOB0 - PB27\n 9 SCLK - PA27\n10 MISO - PA25"
- note removed: "P2 Pinout Einsy 2560\n 1 +5V (Now PC5)\n 2 GND\n 3 nRESET\n 4 RX3 - PJ0\n 5 MOSI - PB2\n 6 TX3 - PJ1\n 7 SS - PB0\n 8 PJ2\n 9 SCK - PB1\n10 PH2"
- moved on the sheet: C3, C4, C5, R5, Z1A
